File: adc.kicad_sch (KiCad schematic)
At the start: 38 parts, among them J10 RCA Female, Q10 2N3904, Q11 2N6426, Q12 2N3904, Q13 2N3904, Q14 2N3906, Q8 2N3904, Q9 2N3904, U7 MC10321P

Commit message: added bom exclusions for non mod components
Parts:
- C31, C35, C43, C47, C48, C51, C52, C53, C54, D10, D7, D8, D9, J10, L1, Q10, Q11, Q12, Q13, Q14, Q8, Q9, R54, R55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: now left out of the parts list
