File: audio_io.kicad_sch (KiCad schematic)
At the start: 51 parts, among them J2 RCA Female, J3 RCA Female, J4 3.5mm TS Jack, J5 RCA Female, J6 RCA Female, J7 RCA Female, J8 RCA Female, U1 MC34074P, U3 MC34074P

Commit message: added bom exclusions for non mod components
Parts:
- C12, C13, C14, C15, C16, C17, C18, C19, C20, C22, C24, C29, C36, J2, J3, J4, J5, J6, J7, J8, R10, R14, R15, R16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: now left out of the parts list
