File: dac.kicad_sch (KiCad schematic)
At the start: 28 parts, among them J9 RCA Female, Q15 2N3906, Q16 2N3904, U8 MC10322P

Commit message: added bom exclusions for non mod components
Parts:
- C45, C46, C49, C50, C55, C56, C57, C58, D11, D12, J9, L2, Q15, Q16, R66, R67, R68, R69, R77, R78, R81, R82, R83, R84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: now left out of the parts list
