File: front_panel.kicad_sch (KiCad schematic)
At the start: 11 parts

Commit message: added bom exclusions for non mod components
Parts:
- C10, JP1, RV1, RV2, RV3, RV4, RV5, RV6, RV7, RV8, RV9: now left out of the parts list
Changed lines of the file:
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@@
   )
   (symbol (lib_id "Device:R_Potentiometer") (at 190.5 120.65 0) (unit 1)
-    (in_bom yes) (on_board no)
+    (in_bom no) (on_board no)
     (property "Reference" "RV6" (id 0) (at 186.055 120.65 90))
     (property "Value" "10k Linear Slide" (id 1) (at 187.96 120.65 90))
@@
   )
   (symbol (lib_id "Device:C") (at 74.93 59.69 0) (unit 1)
-    (in_bom yes) (on_board no) (fields_autoplaced)
+    (in_bom no) (on_board no) (fields_autoplaced)
     (property "Reference" "C10" (id 0) (at 77.851 58.8553 0)
       (effects (font (size 1.27 1.27)) (justify left))
@@
   )
   (symbol (lib_id "Device:R_Potentiometer") (at 215.9 120.65 0) (unit 1)
-    (in_bom yes) (on_board no)
+    (in_bom no) (on_board no)
     (property "Reference" "RV7" (id 0) (at 211.455 120.65 90))
     (property "Value" "10k Linear Slide" (id 1) (at 213.36 120.65 90))
@@
   )
   (symbol (lib_id "power:GND") (at 139.7 66.04 0) (unit 1)
-    (in_bom yes) (on_board no) (fields_autoplaced)
+    (in_bom no) (on_board no) (fields_autoplaced)
     (property "Reference" "#PWR0191" (id 0) (at 139.7 72.39 0)
       (effects (font (size 1.27 1.27)) hide)
@@
   )
   (symbol (lib_id "Device:R_Potentiometer") (at 114.3 120.65 0) (unit 1)
-    (in_bom yes) (on_board no)
+    (in_bom no) (on_board no)
     (property "Reference" "RV3" (id 0) (at 109.855 120.65 90))
     (property "Value" "10k Linear Slide" (id 1) (at 111.76 120.65 90))
@@
   )
   (symbol (lib_id "Device:R_Potentiometer_Dual") (at 26.67 167.64 270) (unit 1)
-    (in_bom yes) (on_board no)
+    (in_bom no) (on_board no)
     (property "Reference" "RV1" (id 0) (at 20.32 167.64 0))
     (property "Value" "10k Linear Dual-Slide" (id 1) (at 18.5467 167.64 0))
@@
   )
   (symbol (lib_id "Device:R_Potentiometer") (at 241.3 120.65 0) (unit 1)
-    (in_bom yes) (on_board no)
+    (in_bom no) (on_board no)
     (property "Reference" "RV8" (id 0) (at 236.855 120.65 90))
     (property "Value" "10k Linear Slide" (id 1) (at 238.76 120.65 90))
@@
   )
   (symbol (lib_id "Videonics Proceessor Plus:R_Potentiometer_With_Switch") (at 67.31 120.65 0) (unit 1)
-    (in_bom yes) (on_board no)
+    (in_bom no) (on_board no)
     (property "Reference" "RV2" (id 0) (at 58.42 119.38 0))
     (property "Value" "8k Linear" (id 1) (at 58.42 121.92 0))
@@
   )
   (symbol (lib_id "Connector_Generic:Conn_02x13_Odd_Even") (at 207.01 63.5 0) (unit 1)
-    (in_bom yes) (on_board no) (fields_autoplaced)
+    (in_bom no) (on_board no) (fields_autoplaced)
     (property "Reference" "JP1" (id 0) (at 208.28 45.8272 0))
     (property "Value" "Conn_02x13_Odd_Even" (id 1) (at 208.28 45.8271 0)
@@
   )
   (symbol (lib_id "Device:R_Potentiometer") (at 139.7 120.65 0) (unit 1)
-    (in_bom yes) (on_board no)
+    (in_bom no) (on_board no)
     (property "Reference" "RV4" (id 0) (at 135.255 120.65 90))
     (property "Value" "10k Linear Slide" (id 1) (at 137.16 120.65 90))
@@
   )
   (symbol (lib_id "Device:R_Potentiometer") (at 266.7 120.65 0) (unit 1)
-    (in_bom yes) (on_board no)
+    (in_bom no) (on_board no)
     (property "Reference" "RV9" (id 0) (at 262.255 120.65 90))
     (property "Value" "10k Linear Slide" (id 1) (at 264.16 120.65 90))
@@
   )
   (symbol (lib_id "power:+10V") (at 74.93 49.53 0) (unit 1)
-    (in_bom yes) (on_board no) (fields_autoplaced)
+    (in_bom no) (on_board no) (fields_autoplaced)
     (property "Reference" "#PWR0138" (id 0) (at 74.93 53.34 0)
       (effects (font (size 1.27 1.27)) hide)
@@
   )
   (symbol (lib_id "power:GND") (at 74.93 66.04 0) (unit 1)
-    (in_bom yes) (on_board no) (fields_autoplaced)
+    (in_bom no) (on_board no) (fields_autoplaced)
     (property "Reference" "#PWR0134" (id 0) (at 74.93 72.39 0)
       (effects (font (size 1.27 1.27)) hide)
@@
   )
   (symbol (lib_id "Device:R_Potentiometer") (at 165.1 120.65 0) (unit 1)
-    (in_bom yes) (on_board no)
+    (in_bom no) (on_board no)
     (property "Reference" "RV5" (id 0) (at 160.655 120.65 90))
     (property "Value" "10k Linear Slide" (id 1) (at 162.56 120.65 90))
