File: multiplexer.kicad_sch (KiCad schematic)
At the start: 18 parts, among them Q1 2N3906, Q2 2N3906, Q3 2N3906, U2 MC14067BDW

Commit message: added bom exclusions for non mod components
Parts:
- C11, C26, PATCH_C1, Q1, Q2, Q3, R11, R12, R13, R21, R22, R23, R24, R25, R26, R27, R29, U2: now left out of the parts list
Changed lines of the file:
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@@
   )
   (symbol (lib_id "power:GND") (at 213.36 119.38 0) (mirror y) (unit 1)
-    (in_bom yes) (on_board no) (fields_autoplaced)
+    (in_bom no) (on_board no) (fields_autoplaced)
     (property "Reference" "#PWR0152" (id 0) (at 213.36 125.73 0)
       (effects (font (size 1.27 1.27)) hide)
@@
   )
   (symbol (lib_id "power:GND") (at 92.71 123.19 0) (unit 1)
-    (in_bom yes) (on_board no) (fields_autoplaced)
+    (in_bom no) (on_board no) (fields_autoplaced)
     (property "Reference" "#PWR0137" (id 0) (at 92.71 129.54 0)
       (effects (font (size 1.27 1.27)) hide)
@@
   )
   (symbol (lib_id "power:+5V") (at 55.88 74.93 0) (unit 1)
-    (in_bom yes) (on_board no) (fields_autoplaced)
+    (in_bom no) (on_board no) (fields_autoplaced)
     (property "Reference" "#PWR0113" (id 0) (at 55.88 78.74 0)
       (effects (font (size 1.27 1.27)) hide)
@@
   )
   (symbol (lib_id "power:+5V") (at 252.73 36.83 0) (mirror y) (unit 1)
-    (in_bom yes) (on_board no) (fields_autoplaced)
+    (in_bom no) (on_board no) (fields_autoplaced)
     (property "Reference" "#PWR0148" (id 0) (at 252.73 40.64 0)
       (effects (font (size 1.27 1.27)) hide)
@@
   )
   (symbol (lib_id "Device:C") (at 66.04 95.25 0) (unit 1)
-    (in_bom yes) (on_board no) (fields_autoplaced)
+    (in_bom no) (on_board no) (fields_autoplaced)
     (property "Reference" "C26" (id 0) (at 68.961 94.4153 0)
       (effects (font (size 1.27 1.27)) (justify left))
@@
   )
   (symbol (lib_id "power:+5V") (at 198.12 36.83 0) (mirror y) (unit 1)
-    (in_bom yes) (on_board no) (fields_autoplaced)
+    (in_bom no) (on_board no) (fields_autoplaced)
     (property "Reference" "#PWR0149" (id 0) (at 198.12 40.64 0)
       (effects (font (size 1.27 1.27)) hide)
@@
   )
   (symbol (lib_id "Device:C_Polarized_US") (at 92.71 116.84 0) (unit 1)
-    (in_bom yes) (on_board no) (fields_autoplaced)
+    (in_bom no) (on_board no) (fields_autoplaced)
     (property "Reference" "PATCH_C1" (id 0) (at 95.631 115.3703 0)
       (effects (font (size 1.27 1.27)) (justify left))
@@
   )
   (symbol (lib_id "Transistor_BJT:2N3906") (at 58.42 90.17 180) (unit 1)
-    (in_bom yes) (on_board no) (fields_autoplaced)
+    (in_bom no) (on_board no) (fields_autoplaced)
     (property "Reference" "Q3" (id 0) (at 53.5687 89.3353 0)
       (effects (font (size 1.27 1.27)) (justify left))
@@
   )
   (symbol (lib_id "Device:R") (at 259.08 54.61 270) (mirror x) (unit 1)
-    (in_bom yes) (on_board no) (fields_autoplaced)
+    (in_bom no) (on_board no) (fields_autoplaced)
     (property "Reference" "R13" (id 0) (at 259.08 49.8942 90))
     (property "Value" "6.8k" (id 1) (at 259.08 52.4311 90))
@@
   )
   (symbol (lib_id "Transistor_BJT:2N3906") (at 191.77 54.61 180) (unit 1)
-    (in_bom yes) (on_board no) (fields_autoplaced)
+    (in_bom no) (on_board no) (fields_autoplaced)
     (property "Reference" "Q1" (id 0) (at 186.9186 53.7753 0)
       (effects (font (size 1.27 1.27)) (justify left))
@@
   )
   (symbol (lib_id "Device:R") (at 204.47 54.61 270) (mirror x) (unit 1)
-    (in_bom yes) (on_board no) (fields_autoplaced)
+    (in_bom no) (on_board no) (fields_autoplaced)
     (property "Reference" "R11" (id 0) (at 204.47 49.8942 90))
     (property "Value" "6.8k" (id 1) (at 204.47 52.4311 90))
@@
   )
   (symbol (lib_id "Device:R") (at 243.84 43.18 0) (mirror y) (unit 1)
-    (in_bom yes) (on_board no) (fields_autoplaced)
+    (in_bom no) (on_board no) (fields_autoplaced)
     (property "Reference" "R23" (id 0) (at 242.062 42.3453 0)
       (effects (font (size 1.27 1.27)) (justify left))
@@
   )
   (symbol (lib_id "Videonics Proceessor Plus:MC14067BDW") (at 129.54 92.71 0) (unit 1)
-    (in_bom yes) (on_board no) (fields_autoplaced)
+    (in_bom no) (on_board no) (fields_autoplaced)
     (property "Reference" "U2" (id 0) (at 129.54 63.5322 0))
     (property "Value" "MC14067BDW" (id 1) (at 129.54 66.0691 0))
@@
   )
   (symbol (lib_id "Device:R") (at 205.74 90.17 0) (mirror y) (unit 1)
-    (in_bom yes) (on_board no) (fields_autoplaced)
+    (in_bom no) (on_board no) (fields_autoplaced)
     (property "Reference" "R26" (id 0) (at 207.518 89.3353 0)
       (effects (font (size 1.27 1.27)) (justify right))
@@
   )
   (symbol (lib_id "power:+5V") (at 149.86 67.31 0) (unit 1)
-    (in_bom yes) (on_board no) (fields_autoplaced)
+    (in_bom no) (on_board no) (fields_autoplaced)
     (property "Reference" "#PWR0109" (id 0) (at 149.86 71.12 0)
       (effects (font (size 1.27 1.27)) hide)
@@
   )
   (symbol (lib_id "Device:R") (at 213.36 113.03 0) (mirror y) (unit 1)
-    (in_bom yes) (on_board no) (fields_autoplaced)
+    (in_bom no) (on_board no) (fields_autoplaced)
     (property "Reference" "R12" (id 0) (at 211.582 112.1953 0)
       (effects (font (size 1.27 1.27)) (justify left))
@@
   )
   (symbol (lib_id "Device:R") (at 198.12 43.18 0) (mirror y) (unit 1)
-    (in_bom yes) (on_board no) (fields_autoplaced)
+    (in_bom no) (on_board no) (fields_autoplaced)
     (property "Reference" "R22" (id 0) (at 196.342 42.3453 0)
       (effects (font (size 1.27 1.27)) (justify left))
@@
   )
   (symbol (lib_id "power:GND") (at 149.86 115.57 0) (unit 1)
-    (in_bom yes) (on_board no) (fields_autoplaced)
+    (in_bom no) (on_board no) (fields_autoplaced)
     (property "Reference" "#PWR0110" (id 0) (at 149.86 121.92 0)
       (effects (font (size 1.27 1.27)) hide)
@@
   )
   (symbol (lib_id "power:GND") (at 106.68 85.09 0) (unit 1)
-    (in_bom yes) (on_board no)
+    (in_bom no) (on_board no)
     (property "Reference" "#PWR0112" (id 0) (at 106.68 91.44 0)
       (effects (font (size 1.27 1.27)) hide)
@@
   )
   (symbol (lib_id "Device:R") (at 189.23 43.18 0) (mirror y) (unit 1)
-    (in_bom yes) (on_board no) (fields_autoplaced)
+    (in_bom no) (on_board no) (fields_autoplaced)
     (property "Reference" "R21" (id 0) (at 187.452 42.3453 0)
       (effects (font (size 1.27 1.27)) (justify left))
@@
   )
   (symbol (lib_id "Device:R") (at 55.88 80.01 0) (unit 1)
-    (in_bom yes) (on_board no) (fields_autoplaced)
+    (in_bom no) (on_board no) (fields_autoplaced)
     (property "Reference" "R29" (id 0) (at 57.658 79.1753 0)
       (effects (font (size 1.27 1.27)) (justify left))
@@
   )
   (symbol (lib_id "power:+5V") (at 142.24 137.16 0) (unit 1)
-    (in_bom yes) (on_board no) (fields_autoplaced)
+    (in_bom no) (on_board no) (fields_autoplaced)
     (property "Reference" "#PWR0151" (id 0) (at 142.24 140.97 0)
       (effects (font (size 1.27 1.27)) hide)
@@
   )
   (symbol (lib_id "power:GND") (at 149.86 82.55 0) (unit 1)
-    (in_bom yes) (on_board no) (fields_autoplaced)
+    (in_bom no) (on_board no) (fields_autoplaced)
     (property "Reference" "#PWR0150" (id 0) (at 149.86 88.9 0)
       (effects (font (size 1.27 1.27)) hide)
@@
   )
   (symbol (lib_id "Device:C") (at 149.86 76.2 0) (unit 1)
-    (in_bom yes) (on_board no) (fields_autoplaced)
+    (in_bom no) (on_board no) (fields_autoplaced)
     (property "Reference" "C11" (id 0) (at 152.781 75.3653 0)
       (effects (font (size 1.27 1.27)) (justify left))
@@
   )
   (symbol (lib_id "power:GND") (at 66.04 100.33 0) (unit 1)
-    (in_bom yes) (on_board no) (fields_autoplaced)
+    (in_bom no) (on_board no) (fields_autoplaced)
     (property "Reference" "#PWR0111" (id 0) (at 66.04 106.68 0)
       (effects (font (size 1.27 1.27)) hide)
@@
   )
   (symbol (lib_id "Device:R") (at 196.85 90.17 0) (mirror y) (unit 1)
-    (in_bom yes) (on_board no) (fields_autoplaced)
+    (in_bom no) (on_board no) (fields_autoplaced)
     (property "Reference" "R24" (id 0) (at 198.628 89.3353 0)
       (effects (font (size 1.27 1.27)) (justify right))
@@
   )
   (symbol (lib_id "Transistor_BJT:2N3906") (at 246.38 54.61 180) (unit 1)
-    (in_bom yes) (on_board no) (fields_autoplaced)
+    (in_bom no) (on_board no) (fields_autoplaced)
     (property "Reference" "Q2" (id 0) (at 241.5286 53.7753 0)
       (effects (font (size 1.27 1.27)) (justify left))
@@
   )
   (symbol (lib_id "Device:R") (at 142.24 143.51 0) (unit 1)
-    (in_bom yes) (on_board no) (fields_autoplaced)
+    (in_bom no) (on_board no) (fields_autoplaced)
     (property "Reference" "R27" (id 0) (at 144.018 142.6753 0)
       (effects (font (size 1.27 1.27)) (justify left))
@@
   )
   (symbol (lib_id "Device:R") (at 252.73 43.18 0) (mirror y) (unit 1)
-    (in_bom yes) (on_board no) (fields_autoplaced)
+    (in_bom no) (on_board no) (fields_autoplaced)
     (property "Reference" "R25" (id 0) (at 250.952 42.3453 0)
       (effects (font (size 1.27 1.27)) (justify left))
