File: power_supply.kicad_sch (KiCad schematic)
At the start: 25 parts, among them P1 12VAC

Commit message: added bom exclusions for non mod components
Parts:
- C1, C2, C27, C3, C38, C4, C41, C44, C5, C59, C6, C60, C7, C8, C9, D1, D2, D3, D4, P1, PATCH_D1, R1, VR1, VR2: now left out of the parts list
