File: video_processor.kicad_sch (KiCad schematic)
At the start: 29 parts, among them Q4 2N3904, Q5 2N3906, U6 AMI_9128MAB_P, Y1 RXD MP49 14.31818

Commit message: cleanup and rename subsheets, increment rev
Other:
- title: Video Processor -> Video Processor (DSP)
Changed lines of the file:
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@@
   (paper "A4")
   (title_block
-    (title "Video Processor")
-    (date "2023-05-24")
-    (rev "3")
+    (title "Video Processor (DSP)")
+    (date "2023-07-19")
+    (rev "4")
   )
   (junction (at 241.3 118.11) (diameter 0) (color 0 0 0 0)

Commit message: added bom exclusions for non mod components
Parts:
- BLEV0, BLEV1, C28, C30, C32, C33, C34, C37, C42, CVC01, D6, PATCH_C2, PATCH_R1, Q4, Q5, R37, R38, R39, R40, R41, R42, R43, R51, R52, R53, R87, R88, U6, Y1: now left out of the parts list
