File: datbusbuffer.kicad_sch (KiCad schematic)
At the start: 9 parts, among them J11 DAT_MCU, Q17 2N3904, U13 74LS241, U14 74LS241

Commit message: Minor formatting updates
Connections:
- net +5V: now also U14.15 (I2b), U14.17 (I3b), U14.3 (O3b), U14.5 (O2b)
- no-connect marks 4 -> 0
Changed lines of the file:
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@@
 (kicad_sch (version 20211123) (generator eeschema)
   (paper "A4")
+  (junction (at 214.63 66.04) (diameter 0) (color 0 0 0 0)
+  )
+  (junction (at 186.69 66.04) (diameter 0) (color 0 0 0 0)
+  )
   (junction (at 110.49 96.52) (diameter 0) (color 0 0 0 0)
   )
@@
   (junction (at 87.63 96.52) (diameter 0) (color 0 0 0 0)
   )
-  (no_connect (at 187.96 67.31))
-  (no_connect (at 213.36 67.31))
-  (no_connect (at 187.96 64.77))
-  (no_connect (at 213.36 64.77))
   (bus_entry (at 48.26 142.24) (size 2.54 2.54)
     (stroke (width 0) (type default) (color 0 0 0 0))
@@
     (stroke (width 0) (type default) (color 0 0 0 0))
   )
+  (wire (pts (xy 186.69 66.04) (xy 186.69 67.31))
+    (stroke (width 0) (type default) (color 0 0 0 0))
+  )
   (bus (pts (xy 48.26 132.08) (xy 48.26 134.62))
     (stroke (width 0) (type default) (color 0 0 0 0))
@@
     (stroke (width 0) (type default) (color 0 0 0 0))
   )
+  (wire (pts (xy 186.69 67.31) (xy 187.96 67.31))
+    (stroke (width 0) (type default) (color 0 0 0 0))
+  )
+  (wire (pts (xy 186.69 64.77) (xy 186.69 66.04))
+    (stroke (width 0) (type default) (color 0 0 0 0))
+  )
   (wire (pts (xy 50.8 142.24) (xy 66.04 142.24))
     (stroke (width 0) (type default) (color 0 0 0 0))
@@
     (stroke (width 0) (type default) (color 0 0 0 0))
   )
+  (wire (pts (xy 214.63 64.77) (xy 214.63 66.04))
+    (stroke (width 0) (type default) (color 0 0 0 0))
+  )
   (wire (pts (xy 124.46 82.55) (xy 124.46 83.82))
     (stroke (width 0) (type default) (color 0 0 0 0))
@@
     (stroke (width 0) (type default) (color 0 0 0 0))
   )
+  (wire (pts (xy 214.63 67.31) (xy 213.36 67.31))
+    (stroke (width 0) (type default) (color 0 0 0 0))
+  )
   (wire (pts (xy 176.53 49.53) (xy 187.96 49.53))
     (stroke (width 0) (type default) (color 0 0 0 0))
   )
+  (wire (pts (xy 185.42 66.04) (xy 186.69 66.04))
+    (stroke (width 0) (type default) (color 0 0 0 0))
+  )
   (wire (pts (xy 213.36 49.53) (xy 224.79 49.53))
     (stroke (width 0) (type default) (color 0 0 0 0))
@@
     (stroke (width 0) (type default) (color 0 0 0 0))
   )
+  (wire (pts (xy 214.63 66.04) (xy 214.63 67.31))
+    (stroke (width 0) (type default) (color 0 0 0 0))
+  )
   (wire (pts (xy 107.95 72.39) (xy 111.76 72.39))
     (stroke (width 0) (type default) (color 0 0 0 0))
@@
     (stroke (width 0) (type default) (color 0 0 0 0))
   )
+  (wire (pts (xy 213.36 64.77) (xy 214.63 64.77))
+    (stroke (width 0) (type default) (color 0 0 0 0))
+  )
   (wire (pts (xy 248.92 90.17) (xy 248.92 92.71))
     (stroke (width 0) (type default) (color 0 0 0 0))
@@
     (stroke (width 0) (type default) (color 0 0 0 0))
   )
+  (wire (pts (xy 187.96 64.77) (xy 186.69 64.77))
+    (stroke (width 0) (type default) (color 0 0 0 0))
+  )
   (wire (pts (xy 50.8 149.86) (xy 66.04 149.86))
     (stroke (width 0) (type default) (color 0 0 0 0))
@@
   )
   (wire (pts (xy 50.8 132.08) (xy 66.04 132.08))
+    (stroke (width 0) (type default) (color 0 0 0 0))
+  )
+  (wire (pts (xy 214.63 66.04) (xy 215.9 66.04))
     (stroke (width 0) (type default) (color 0 0 0 0))
   )
@@
   (hierarchical_label "DAT_DSP[1..14]" (shape output) (at 245.11 124.46 0)
     (effects (font (size 1.27 1.27)) (justify left))
+  )
+  (symbol (lib_id "power:+5V") (at 185.42 66.04 90) (unit 1)
+    (in_bom yes) (on_board yes) (fields_autoplaced)
+    (property "Reference" "#PWR?" (id 0) (at 189.23 66.04 0)
+      (effects (font (size 1.27 1.27)) hide)
+    )
+    (property "Value" "+5V" (id 1) (at 182.2451 66.4738 90)
+      (effects (font (size 1.27 1.27)) (justify left))
+    )
+    (property "Footprint" "" (id 2) (at 185.42 66.04 0)
+      (effects (font (size 1.27 1.27)) hide)
+    )
+    (property "Datasheet" "" (id 3) (at 185.42 66.04 0)
+      (effects (font (size 1.27 1.27)) hide)
+    )
+    (pin "1")
   )
   (symbol (lib_id "power:GND") (at 200.66 83.82 0) (unit 1)
@@
     (pin "3")
   )
+  (symbol (lib_id "power:+5V") (at 215.9 66.04 270) (unit 1)
+    (in_bom yes) (on_board yes) (fields_autoplaced)
+    (property "Reference" "#PWR?" (id 0) (at 212.09 66.04 0)
+      (effects (font (size 1.27 1.27)) hide)
+    )
+    (property "Value" "+5V" (id 1) (at 219.075 66.4738 90)
+      (effects (font (size 1.27 1.27)) (justify left))
+    )
+    (property "Footprint" "" (id 2) (at 215.9 66.04 0)
+      (effects (font (size 1.27 1.27)) hide)
+    )
+    (property "Datasheet" "" (id 3) (at 215.9 66.04 0)
+      (effects (font (size 1.27 1.27)) hide)
+    )
+    (pin "1")
+  )
   (symbol (lib_id "power:+5V") (at 124.46 40.64 0) (unit 1)

Commit message: smaller resistor footprint
Parts:
- R92, R93, R94: footprint Resistor_THT:R_Axial_DIN0207_L6.3mm_D2.5mm_P10.16mm_Horizontal -> Resistor_THT:R_Axial_DIN0207_L6.3mm_D2.5mm_P2.54mm_Vertical
Changed lines of the file:
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@@
       (effects (font (size 1.27 1.27)) (justify left))
     )
-    (property "Footprint" "Resistor_THT:R_Axial_DIN0207_L6.3mm_D2.5mm_P10.16mm_Horizontal" (id 2) (at 85.852 91.44 90)
+    (property "Footprint" "Resistor_THT:R_Axial_DIN0207_L6.3mm_D2.5mm_P2.54mm_Vertical" (id 2) (at 85.852 91.44 90)
       (effects (font (size 1.27 1.27)) hide)
     )
@@
     (property "Reference" "R93" (id 0) (at 73.66 98.1542 90))
     (property "Value" "1k" (id 1) (at 73.66 100.6911 90))
-    (property "Footprint" "Resistor_THT:R_Axial_DIN0207_L6.3mm_D2.5mm_P10.16mm_Horizontal" (id 2) (at 73.66 104.648 90)
+    (property "Footprint" "Resistor_THT:R_Axial_DIN0207_L6.3mm_D2.5mm_P2.54mm_Vertical" (id 2) (at 73.66 104.648 90)
       (effects (font (size 1.27 1.27)) hide)
     )
@@
       (effects (font (size 1.27 1.27)) (justify left))
     )
-    (property "Footprint" "Resistor_THT:R_Axial_DIN0207_L6.3mm_D2.5mm_P10.16mm_Horizontal" (id 2) (at 61.722 107.95 90)
-      (effects (font (size 1.27 1.27)) hide)
-    )
+    (property "Footprint" "Resistor_THT:R_Axial_DIN0207_L6.3mm_D2.5mm_P2.54mm_Vertical" (id 2) (at 61.722 107.95 90)
+      (effects (font (size 1.27 1.27)) hide)
+    )

Commit message: schematic updated
Parts:
- removed Q17: 2N3904, Package_TO_SOT_THT:TO-92_Inline_Wide, symbol Transistor_BJT:2N3904
- removed R93: 1k, Resistor_THT:R_Axial_DIN0207_L6.3mm_D2.5mm_P2.54mm_Vertical, symbol Device:R
- removed R94: 10k, Resistor_THT:R_Axial_DIN0207_L6.3mm_D2.5mm_P2.54mm_Vertical, symbol Device:R
- removed U13, U14: 74LS241, Package_DIP:DIP-20_W7.62mm, symbol 74xx:74LS241
- added U14, U15: 74LS244, symbol 74xx:74LS244
- R92: footprint Resistor_THT:R_Axial_DIN0207_L6.3mm_D2.5mm_P2.54mm_Vertical -> (none)
Connections:
- net +5V: now also U14.20 (VCC), U15.20 (VCC)
- net DAT_DSP1: now also U14.18 (O0a)
- net DAT_DSP10: now also U15.16 (O1a)
- net DAT_DSP11: now also U15.14 (O2a)
- net DAT_DSP12: now also U15.12 (O3a)
- net DAT_DSP13: now also U15.9 (O0b)
- net DAT_DSP14: now also U15.7 (O1b)
- net DAT_DSP2: now also U14.16 (O1a)
- net DAT_DSP3: now also U14.14 (O2a)
- net DAT_DSP4: now also U14.12 (O3a)
- net DAT_DSP5: now also U14.9 (O0b)
- net DAT_DSP6: now also U14.7 (O1b)
- net DAT_DSP7: now also U14.5 (O2b)
- net DAT_DSP8: now also U14.3 (O3b)
- net DAT_DSP9: now also U15.18 (O0a)
- net DAT_MCU1: now also U14.2 (I0a)
- net DAT_MCU10: now also U15.4 (I1a)
- net DAT_MCU11: now also U15.6 (I2a)
- net DAT_MCU12: now also U15.8 (I3a)
- net DAT_MCU13: now also U15.11 (I0b)
- net DAT_MCU14: now also U15.13 (I1b)
- net DAT_MCU2: now also U14.4 (I1a)
- net DAT_MCU3: now also U14.6 (I2a)
- net DAT_MCU4: now also U14.8 (I3a)
- net DAT_MCU5: now also U14.11 (I0b)
- net DAT_MCU6: now also U14.13 (I1b)
- net DAT_MCU7: now also U14.15 (I2b)
- net DAT_MCU8: now also U14.17 (I3b)
- net DAT_MCU9: now also U15.2 (I0a)
- net GND: now also U14.10 (GND), U15.10 (GND), U15.15 (I2b), U15.17 (I3b), U15.3 (O3b), U15.5 (O2b)
- net ~{DAT_BUF_OE}: now also U14.1 (OEa), U14.19 (OEb), U15.1 (OEa), U15.19 (OEb)

Commit message: assigned footprints
Parts:
- R92: footprint (none) -> Resistor_THT:R_Axial_DIN0207_L6.3mm_D2.5mm_P2.54mm_Vertical
- U14, U15: footprint (none) -> Package_DIP:DIP-20_W7.62mm
Changed lines of the file:
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@@
       (effects (font (size 1.27 1.27)) (justify left))
     )
-    (property "Footprint" "" (id 2) (at 124.46 62.23 0)
+    (property "Footprint" "Package_DIP:DIP-20_W7.62mm" (id 2) (at 124.46 62.23 0)
       (effects (font (size 1.27 1.27)) hide)
     )
@@
       (effects (font (size 1.27 1.27)) (justify left))
     )
-    (property "Footprint" "" (id 2) (at 200.66 62.23 0)
+    (property "Footprint" "Package_DIP:DIP-20_W7.62mm" (id 2) (at 200.66 62.23 0)
       (effects (font (size 1.27 1.27)) hide)
     )
@@
       (effects (font (size 1.27 1.27)) (justify left))
     )
-    (property "Footprint" "" (id 2) (at 78.232 78.74 90)
+    (property "Footprint" "Resistor_THT:R_Axial_DIN0207_L6.3mm_D2.5mm_P2.54mm_Vertical" (id 2) (at 78.232 78.74 90)
       (effects (font (size 1.27 1.27)) hide)
     )
