File: sc403860p.kicad_sch (KiCad schematic)
At the start: 20 parts, among them J1 3.5mm TS Jack, Q6 2N3904, Q7 2N3904, U4 74LS221, U5 SC403860P

Commit message: cleanup and rename subsheets, increment rev
Other:
- note added: "RS232 UART or GPI UART: 19200 baud, 1 start, 1 stop Functionality not documented by manufacturer"
- note removed: "RS232 UART or GPI UART: 19200 baud, 1 start, 1 stop"
- title: Device Settings Processor -> Setting Controller (MCU)
Changed lines of the file:
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@@
   (paper "A4")
   (title_block
-    (title "Device Settings Processor")
-    (date "2023-05-24")
-    (rev "3")
+    (title "Setting Controller (MCU)")
+    (date "2023-07-19")
+    (rev "4")
   )
   (junction (at 146.05 147.32) (diameter 0) (color 0 0 0 0)
@@
     (stroke (width 0) (type default) (color 0 0 0 0))
   )
+  (wire (pts (xy 123.19 77.47) (xy 153.67 77.47))
+    (stroke (width 0) (type default) (color 0 0 0 0))
+  )
+  (wire (pts (xy 146.05 142.24) (xy 146.05 147.32))
+    (stroke (width 0) (type default) (color 0 0 0 0))
+  )
+  (wire (pts (xy 146.05 147.32) (xy 146.05 148.59))
+    (stroke (width 0) (type default) (color 0 0 0 0))
+  )
+  (wire (pts (xy 110.49 90.17) (xy 123.19 90.17))
+    (stroke (width 0) (type default) (color 0 0 0 0))
+  )
+  (wire (pts (xy 40.64 82.55) (xy 52.07 82.55))
+    (stroke (width 0) (type default) (color 0 0 0 0))
+  )
+  (wire (pts (xy 40.64 77.47) (xy 52.07 77.47))
+    (stroke (width 0) (type default) (color 0 0 0 0))
+  )
+  (wire (pts (xy 223.52 118.11) (xy 223.52 120.65))
+    (stroke (width 0) (type default) (color 0 0 0 0))
+  )
+  (wire (pts (xy 121.92 170.18) (xy 121.92 171.45))
+    (stroke (width 0) (type default) (color 0 0 0 0))
+  )
+  (bus (pts (xy 124.46 104.14) (xy 133.35 104.14))
+    (stroke (width 0) (type default) (color 0 0 0 0))
+  )
+  (wire (pts (xy 110.49 95.25) (xy 121.92 95.25))
+    (stroke (width 0) (type default) (color 0 0 0 0))
+  )
+  (wire (pts (xy 97.79 172.72) (xy 97.79 177.8))
+    (stroke (width 0) (type default) (color 0 0 0 0))
+  )
+  (wire (pts (xy 111.76 138.43) (xy 111.76 137.16))
+    (stroke (width 0) (type default) (color 0 0 0 0))
+  )
   (wire (pts (xy 40.64 67.31) (xy 52.07 67.31))
-    (stroke (width 0) (type default) (color 0 0 0 0))
-  )
-  (wire (pts (xy 123.19 77.47) (xy 153.67 77.47))
-    (stroke (width 0) (type default) (color 0 0 0 0))
-  )
-  (wire (pts (xy 146.05 142.24) (xy 146.05 147.32))
-    (stroke (width 0) (type default) (color 0 0 0 0))
-  )
-  (wire (pts (xy 146.05 147.32) (xy 146.05 148.59))
-    (stroke (width 0) (type default) (color 0 0 0 0))
-  )
-  (wire (pts (xy 110.49 90.17) (xy 123.19 90.17))
-    (stroke (width 0) (type default) (color 0 0 0 0))
-  )
-  (wire (pts (xy 40.64 82.55) (xy 52.07 82.55))
-    (stroke (width 0) (type default) (color 0 0 0 0))
-  )
-  (wire (pts (xy 40.64 77.47) (xy 52.07 77.47))
-    (stroke (width 0) (type default) (color 0 0 0 0))
-  )
-  (wire (pts (xy 223.52 118.11) (xy 223.52 120.65))
-    (stroke (width 0) (type default) (color 0 0 0 0))
-  )
-  (wire (pts (xy 121.92 170.18) (xy 121.92 171.45))
-    (stroke (width 0) (type default) (color 0 0 0 0))
-  )
-  (bus (pts (xy 124.46 104.14) (xy 133.35 104.14))
-    (stroke (width 0) (type default) (color 0 0 0 0))
-  )
-  (wire (pts (xy 110.49 95.25) (xy 121.92 95.25))
-    (stroke (width 0) (type default) (color 0 0 0 0))
-  )
-  (wire (pts (xy 97.79 172.72) (xy 97.79 177.8))
-    (stroke (width 0) (type default) (color 0 0 0 0))
-  )
-  (wire (pts (xy 111.76 138.43) (xy 111.76 137.16))
     (stroke (width 0) (type default) (color 0 0 0 0))
   )
@@
     (effects (font (size 1.27 1.27)) (justify right bottom))
   )
-  (text "RS232 UART or GPI\nUART: 19200 baud, 1 start, 1 stop"
-    (at 46.99 139.7 0)
+  (text "RS232 UART or GPI\nUART: 19200 baud, 1 start, 1 stop\nFunctionality not documented by manufacturer"
+    (at 40.64 139.7 0)
     (effects (font (size 1.27 1.27)) (justify left bottom))
   )

Commit message: added bom exclusions for non mod components
Parts:
- C21, C23, C25, C39, C40, D5, J1, MCLK1, PAL1, Q6, Q7, R28, R57, R58, R59, R60, R61, R62, U4, U5: now left out of the parts list

Commit message: added vid_blk and fixed inverter on dat 0
Connections:
- net ~{VID_BLK}: now reaches Q7.3 (C), R60.2, U5.33 (Pin_33)
Changed lines of the file:
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@@
   (junction (at 132.08 147.32) (diameter 0) (color 0 0 0 0)
+  )
+  (junction (at 158.75 69.85) (diameter 0) (color 0 0 0 0)
   )
   (junction (at 121.92 171.45) (diameter 0) (color 0 0 0 0)
@@
     (stroke (width 0) (type default) (color 0 0 0 0))
   )
+  (wire (pts (xy 158.75 69.85) (xy 163.83 69.85))
+    (stroke (width 0) (type default) (color 0 0 0 0))
+  )
   (wire (pts (xy 208.28 128.27) (xy 208.28 130.81))
     (stroke (width 0) (type default) (color 0 0 0 0))
@@
     (stroke (width 0) (type default) (color 0 0 0 0))
   )
-  (wire (pts (xy 166.37 69.85) (xy 166.37 171.45))
+  (wire (pts (xy 158.75 69.85) (xy 158.75 171.45))
     (stroke (width 0) (type default) (color 0 0 0 0))
   )
@@
     (stroke (width 0) (type default) (color 0 0 0 0))
   )
-  (wire (pts (xy 110.49 69.85) (xy 166.37 69.85))
+  (wire (pts (xy 110.49 69.85) (xy 158.75 69.85))
     (stroke (width 0) (type default) (color 0 0 0 0))
   )
@@
     (stroke (width 0) (type default) (color 0 0 0 0))
   )
-  (wire (pts (xy 166.37 171.45) (xy 121.92 171.45))
+  (wire (pts (xy 158.75 171.45) (xy 121.92 171.45))
     (stroke (width 0) (type default) (color 0 0 0 0))
   )
@@
     (effects (font (size 1.27 1.27)) (justify right))
   )
+  (hierarchical_label "~{VID_BLK}" (shape output) (at 163.83 69.85 0)
+    (effects (font (size 1.27 1.27)) (justify left))
+  )
   (hierarchical_label "MCLK" (shape input) (at 119.38 54.61 0)
